Commit message: working code for dynamixel motor

File: src/dynamixel_description/urdf/dynamixel.xacro (robot description, xacro)
@@ -44,5 +44,5 @@
   </collision>
 </link>
-<joint name="Revolute 1" type="continuous">
+<joint name="rev_1" type="continuous">
   <origin xyz="0.0 -0.0001 0.0" rpy="0 0 0"/>
   <parent link="base_link"/>

File: src/dynamixel_moveit_config/config/gazebo_dynamixel.urdf (robot description, URDF)
Before this commit: robot dynamixel, 2 links, 1 joints
Joints:
- removed joint Revolute 1
- added joint rev_1: type continuous, parent base_link, child shaft_1, origin xyz=0.0 -0.0001 0.0 rpy=0 0 0, axis 0.0 1.0 0.0

Commit message: major commits of working code

File: src/dynamixel_description/urdf/dynamixel.xacro (robot description, xacro)
@@ -44,6 +44,7 @@
   </collision>
 </link>
-<joint name="rev_1" type="continuous">
+<joint name="rev_1" type="revolute">
   <origin xyz="0.0 -0.0001 0.0" rpy="0 0 0"/>
+  <limit effort="30" lower="0" upper="3.14159265359" velocity="1"/>
   <parent link="base_link"/>
   <child link="shaft_1"/>

File: src/finger_description/urdf/finger.xacro (robot description, xacro)
@@ -84,18 +84,21 @@
   </collision>
 </link>
-<joint name="mcp" type="continuous">
+<joint name="mcp" type="revolute">
   <origin xyz="0.1835 0.04622 0.087809" rpy="0 0 0"/>
+  <limit effort="30" velocity="2" lower="0" upper="1.4"/>
   <parent link="base_link"/>
   <child link="lateral_1"/>
-  <axis xyz="-1.0 0.0 -0.0"/>
+  <axis xyz="1.0 0.0 -0.0"/>
 </joint>
-<joint name="pip" type="continuous">
+<joint name="pip" type="revolute">
   <origin xyz="0.003 0.056752 0.005" rpy="0 0 0"/>
+  <limit effort="30" velocity="2" lower="0" upper="1.4"/>
   <parent link="lateral_1"/>
   <child link="middle_1"/>
   <axis xyz="1.0 0.0 0.0"/>
 </joint>
-<joint name="dip" type="continuous">
+<joint name="dip" type="revolute">
   <origin xyz="0.0 0.051704 4.7e-05" rpy="0 0 0"/>
+  <limit effort="30" velocity="2" lower="0" upper="1.4"/>
   <parent link="middle_1"/>
   <child link="distal_1"/>

File: src/finger_moveit_config/config/gazebo_finger.urdf (robot description, URDF)
Before this commit: robot finger, 4 links, 3 joints
Joints:
- joint mcp: axis -1.0 0.0 -0.0 -> 1.0 0.0 -0.0
